Commit message: integrated gazebo

File: description/robot_core.xacro (robot description, xacro)
@@ -39,4 +39,7 @@
     </xacro:inertial_box>
   </link>
+  <gazebo reference="chassis">
+    <material>Gazebo/White</material>
+  </gazebo>
   <joint name="left_wheel_joint" type="continuous">
     <parent link="base_link" />
@@ -48,10 +51,10 @@
     <visual>
       <geometry>
-        <cylinder length="0.04" radius="0.05" />/> </geometry>
+        <cylinder length="0.04" radius="0.05" /> </geometry>
       <material name="blue" />
     </visual>
     <collision>
       <geometry>
-        <cylinder length="0.04" radius="0.05" />/> </geometry>
+        <cylinder length="0.04" radius="0.05" /> </geometry>
       <material name="blue" />
     </collision>
@@ -69,10 +72,12 @@
     <visual>
       <geometry>
-        <cylinder length="0.04" radius="0.05" />/> </geometry>
+        <cylinder length="0.04" radius="0.05" />
+      </geometry>
       <material name="blue" />
     </visual>
     <collision>
       <geometry>
-        <cylinder length="0.04" radius="0.05" />/> </geometry>
+        <cylinder length="0.04" radius="0.05" />
+      </geometry>
       <material name="blue" />
     </collision>
@@ -103,3 +108,8 @@
     </xacro:inertial_sphere>
   </link>
+  <gazebo reference="caster_wheel">
+    <material>Gazebo/Black</material>
+    <mu1 value="0.001" />
+    <mu2 value="0.001" />
+  </gazebo>
 </robot>

Commit message: added lidar

File: description/robot_core.xacro (robot description, xacro)
@@ -51,10 +51,12 @@
     <visual>
       <geometry>
-        <cylinder length="0.04" radius="0.05" /> </geometry>
+        <cylinder length="0.04" radius="0.05" />
+      </geometry>
       <material name="blue" />
     </visual>
     <collision>
       <geometry>
-        <cylinder length="0.04" radius="0.05" /> </geometry>
+        <cylinder length="0.04" radius="0.05" />
+      </geometry>
       <material name="blue" />
     </collision>
