Commit message: control fixes

File: description/robot.urdf.xacro (robot description, xacro)
@@ -1,7 +1,12 @@
 <?xml version="1.0"?>
 <robot xmlns:xacro="http://www.ros.org/wiki/xacro" name="robot">
+    <xacro:arg name="use_ros2_control" default="true" />
     <xacro:include filename="robot_core.xacro" />
-    <xacro:include filename="ros2_control.xacro" />
-    <!-- <xacro:include filename="gazebo_control.xacro" /> -->
+    <xacro:if value="$(arg use_ros2_control)">
+        <xacro:include filename="ros2_control.xacro" />
+    </xacro:if>
+    <xacro:unless value="$(arg use_ros2_control)">
+        <xacro:include filename="gazebo_control.xacro" />
+    </xacro:unless>
     <!-- <xacro:include filename="lidar.xacro" /> -->
     <!-- <xacro:include filename="camera.xacro" /> -->

File: description/robot_core.xacro (robot description, xacro)
@@ -57,5 +57,5 @@
     <collision>
       <geometry>
-        <cylinder length="0.04" radius="0.05" />
+        <sphere radius="0.05" />
       </geometry>
       <material name="blue" />
@@ -80,5 +80,5 @@
     <collision>
       <geometry>
-        <cylinder length="0.04" radius="0.05" />
+        <sphere radius="0.05" />
       </geometry>
       <material name="blue" />

Commit message: setup slam

File: description/robot.urdf.xacro (robot description, xacro)
@@ -9,6 +9,6 @@
         <xacro:include filename="gazebo_control.xacro" />
     </xacro:unless>
-    <!-- <xacro:include filename="lidar.xacro" /> -->
+    <xacro:include filename="lidar.xacro" />
     <!-- <xacro:include filename="camera.xacro" /> -->
-    <xacro:include filename="depth_camera.xacro" />
+    <!-- <xacro:include filename="depth_camera.xacro" /> -->
 </robot>

File: description/robot_core.xacro (robot description, xacro)
@@ -15,4 +15,11 @@
   </material>
   <link name="base_link">
+  </link>
+  <joint name="base_footprint_joint" type="fixed">
+    <parent link="base_link" />
+    <child link="base_footprint" />
+    <origin xyz="0 0 0" rpy="0 0 0" />
+  </joint>
+  <link name="base_footprint">
   </link>
   <joint name="chassis_joint" type="fixed">
